File: Hardware/BuckBoost/BuckBoost.kicad_sch (KiCad schematic)
At the start: 12 parts, among them J1 Screw_Terminal_01x04, U1 ISL85415FRZ

Commit message: feat: Update PCB
Parts:
- C2, C3: footprint PCM_4ms_Capacitor:C_0603 -> PCM_4ms_Capacitor:CP_Elec_5x5.3
- J1: footprint Connector_PinHeader_2.54mm:PinHeader_1x04_P2.54mm_Vertical -> TerminalBlock_Phoenix:TerminalBlock_Phoenix_PT-1,5-4-3.5-H_1x04_P3.50mm_Horizontal
Changed lines of the file:
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@@
       (effects (font (size 1.27 1.27)) hide)
     )
-    (property "Footprint" "PCM_4ms_Capacitor:C_0603" (at 118.872 107.188 0)
+    (property "Footprint" "PCM_4ms_Capacitor:CP_Elec_5x5.3" (at 118.872 107.188 0)
       (effects (font (size 1.27 1.27)) (justify left) hide)
     )
@@
       (effects (font (size 1.27 1.27)) (justify left))
     )
-    (property "Footprint" "Connector_PinHeader_2.54mm:PinHeader_1x04_P2.54mm_Vertical" (at 88.646 67.818 0)
+    (property "Footprint" "TerminalBlock_Phoenix:TerminalBlock_Phoenix_PT-1,5-4-3.5-H_1x04_P3.50mm_Horizontal" (at 88.646 67.818 0)
       (effects (font (size 1.27 1.27)) hide)
     )
@@
       (effects (font (size 1.27 1.27)) hide)
     )
-    (property "Footprint" "PCM_4ms_Capacitor:C_0603" (at 171.958 106.426 0)
-      (effects (font (size 1.27 1.27)) (justify left) hide)
-    )
+    (property "Footprint" "PCM_4ms_Capacitor:CP_Elec_5x5.3" (at 171.958 106.426 0)
+      (effects (font (size 1.27 1.27)) (justify left) hide)
+    )
